File: KiCAD/VCO_2/VCO_2.kicad_pcb (KiCad board)
At the start: 2 copper layers, 70 x 100 mm, 105 parts, among them J1 MJ-3502, J10 MJ-3502, J11 MJ-3502, J2 MJ-3502, J3 MJ-3502, J4 MJ-3502, J5 MJ-3502, J6 MJ-3502, J7 Power, J8 MJ-3502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

Commit message: updated VCO2
Connections:
- Q1 pad 3: Net-(Q1-Pad1) -> Net-(C5-Pad2)
- Q1 pad 4: Net-(C5-Pad2) -> Net-(Q1-Pad1)
Routing:
- net Net-(C5-Pad2): track 65.8 -> 73.0 mm, vias 2 -> 4
- net Net-(C5-Pad1): track 67.0 -> 69.6 mm
- net Net-(C4-Pad2): track 42.1 -> 41.4 mm
