File: KiCAD/VCO_2/VCO_2.sch (KiCad schematic (older format))
At the start: 84 parts, among them Q1 BC857BS, Q2 MMBFJ112, U1 TL074, U2 TL074, U3 OPA2137, U4 LM311, U5 L78L12_SOT89, U6 L79L12_SOT89

Commit message: updated VCO2
Parts:
- removed Q1: BC857BS, Package_TO_SOT_SMD:SOT-363_SC-70-6, symbol Transistor_BJT:BC857BS
- added Q1: BC847BS, Package_TO_SOT_SMD:SOT-363_SC-70-6, symbol Transistor_BJT:BC847BS
Connections:
- net GND: now also Q1.5 (B2)
- net at D1.2 (A), R13.2, R14.1: now also Q1.2 (B1)
- net at R15.1, R17.1: now also Q1.1 (E1), Q1.4 (E2)
- net at C4.2, R11.1, R16.2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: now also Q1.6 (C1)
- net at C5.2, Q2.2 (D), U2.5 (+): now also Q1.3 (C2)
Changed lines of the file:
@@
 	2350 3400 2350 3350
 Connection ~ 2350 3350
-$Comp
-L Transistor_BJT:BC857BS Q1
-U 1 1 5CCAB607
-P 3025 4000
-F 0 "Q1" H 3200 4100 50  0000 L CNN
-F 1 "BC857BS" H 3225 4000 50  0000 L CNN
-F 2 "Package_TO_SOT_SMD:SOT-363_SC-70-6" H 3225 4100 50  0001 C CNN
-F 3 "https://assets.nexperia.com/documents/data-sheet/BC857BS.pdf" H 3025 4000 50  0001 C CNN
-	1    3025 4000
-	1    0    0    -1
-$EndComp
 Wire Wire Line
 	2350 4000 2700 4000
@@
 	1    0    0    -1
 $EndComp
-$Comp
-L Transistor_BJT:BC857BS Q1
-U 2 1 5CCD5A3F
-P 3775 4000
-F 0 "Q1" H 3925 3900 50  0000 L CNN
-F 1 "BC857BS" H 3975 3850 50  0001 L CNN
-F 2 "Package_TO_SOT_SMD:SOT-363_SC-70-6" H 3975 4100 50  0001 C CNN
-F 3 "https://assets.nexperia.com/documents/data-sheet/BC857BS.pdf" H 3775 4000 50  0001 C CNN
-	2    3775 4000
-	-1   0    0    1
-$EndComp
 Wire Wire Line
 	3125 4375 3675 4375
@@
 Wire Wire Line
 	8225 2300 8225 2500
+$Comp
+L Transistor_BJT:BC847BS Q1
+U 1 1 5CD735AF
+P 3025 4000
+F 0 "Q1" H 3200 4100 50  0000 L CNN
+F 1 "BC847BS" H 3225 3950 50  0000 L CNN
+F 2 "Package_TO_SOT_SMD:SOT-363_SC-70-6" H 3225 4100 50  0001 C CNN
+F 3 "https://assets.nexperia.com/documents/data-sheet/BC847BS.pdf" H 3025 4000 50  0001 C CNN
+	1    3025 4000
+	1    0    0    -1
+$EndComp
+$Comp
+L Transistor_BJT:BC847BS Q1
+U 2 1 5CD77343
+P 3775 4000
+F 0 "Q1" H 3925 4100 50  0000 L CNN
+F 1 "BC847BS" H 3975 3950 50  0001 L CNN
+F 2 "Package_TO_SOT_SMD:SOT-363_SC-70-6" H 3975 4100 50  0001 C CNN
+F 3 "https://assets.nexperia.com/documents/data-sheet/BC847BS.pdf" H 3775 4000 50  0001 C CNN
+	2    3775 4000
+	-1   0    0    -1
+$EndComp
 $EndSCHEMATC
