File: KiCAD/EG/EG.kicad_pcb (KiCad board)
At the start: 2 copper layers, 70 x 45 mm, 44 parts, among them J1 Power, J2 MJ-3502, J3 MJ-3502, Q1 BC847, Q2 BC847, Q3 BC847, Q4 2N7002, U1 TL074, U2 NE555

Commit message: Added RevB and VCA
Parts:
- removed REF** (x4): 1pin, Connectors:1pin
- added CN1: M3_Screw, Synth:M3_Screw_Hole, F.Cu at (65.0, 45.0)
- added CN2: M3_Screw, Synth:M3_Screw_Hole, F.Cu at (65.0, 135.0)
- added CN3: M3_Screw, Synth:M3_Screw_Hole, F.Cu at (95.0, 45.0)
- added CN4: M3_Screw, Synth:M3_Screw_Hole, F.Cu at (95.0, 135.0)
- D1, D2, D3, D4, D5: footprint Diode_SMD:D_SOD-123 -> Synth:D_SOD-123
- D6: footprint LED_THT:LED_D3.0mm -> Synth:LED_D3.0mm_Clear; moved to B.Cu
- J2, J3: value MJ-3502 -> 4832; footprint Connector_PinHeader_2.54mm:PinHeader_1x02_P2.54mm_Vertical -> Synth:Schurter_4832_Jack; moved to B.Cu
- Q1, Q2, Q3, Q4: footprint Package_TO_SOT_SMD:SOT-23 -> TO_SOT_Packages_SMD:SOT-23_Handsoldering
- RV1, RV2, RV3, RV4: footprint Connector_PinHeader_2.54mm:PinHeader_1x03_P2.54mm_Vertical -> Synth:Potentiometer_Bourns_PTV09A-1_Single_Vertical; moved to B.Cu
- moved D6 76.2 mm to (75.0, 121.5)
- moved D5 68.2 mm to (79.7, 121.5)
- moved J3 60.3 mm to (75.0, 130.0), turned to 180 degrees
- moved R8 57.3 mm to (65.4, 93.7)
- moved Q4 56.0 mm to (70.7, 92.5), turned to 270 degrees
- moved R1 55.5 mm to (69.7, 131.2), turned to 270 degrees
- moved R3 54.4 mm to (63.5, 126.9)
- moved R7 54.1 mm to (63.2, 99.6), turned to 90 degrees
- moved R14 52.3 mm to (85.9, 128.4)
- moved RV1 51.8 mm to (80.0, 90.0), turned to 90 degrees
- moved U2 50.9 mm to (67.3, 82.1)
- moved C4 50.8 mm to (67.5, 87.8)
- moved R9 49.1 mm to (80.3, 91.9), turned to 270 degrees
- moved Q2 49.1 mm to (64.8, 115.3), turned to 90 degrees
- moved C5 49.1 mm to (70.1, 73.7), turned to 270 degrees
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Connections:
- net Net-(R10-Pad2) renamed /Release
- net Net-(R11-Pad2) renamed /Attack
- net Net-(R12-Pad1) renamed /Decay
- net Net-(RV1-Pad2) renamed /Sustain
- RV1 pad 1: Net-(R9-Pad2) -> Net-(Q4-Pad3)
- RV1 pad 3: Net-(Q4-Pad3) -> Net-(R9-Pad2)
Routing:
- net EG_Out: track 28.7 -> 68.5 mm, vias 2 -> 3
- net Net-(C6-Pad1): track 30.3 -> 63.0 mm
- net Net-(D3-Pad1): track 4.61 -> 33.1 mm
- net Net-(RV2-Pad1): track 4.04 -> 31.2 mm
- net Net-(C3-Pad2): track 30.5 -> 52.7 mm
- net Net-(D5-Pad2): track 8.70 -> 28.9 mm
- net Gate_In: track 11.3 -> 27.4 mm
- net Net-(Q3-Pad3): track 6.69 -> 22.3 mm
- net Net-(D5-Pad1): track 15.2 -> 28.5 mm
- net ADSR_Out: track 3.70 -> 13.9 mm
- net Net-(Q4-Pad2): track 3.63 -> 11.9 mm
- net /Sustain: track 13.5 -> 21.0 mm
- net +12V: track 17.1 -> 22.3 mm
- net /Release: track 9.78 -> 4.52 mm
- net /Decay: track 4.29 -> 9.53 mm
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Other:
- board size 70 x 45 mm -> 40 x 100 mm
- board text added: "ADSR LEVEL"
- board text added: "ADSR OUTPUT"
- board text added: "ATTACK"
- board text added: "DECAY"
- board text added: "GATE INPUT"
- board text added: "JZK ENVELOPE GENERATOR Rev.B"
- board text added: "RELEASE"
- board text added: "SUSTAIN"
- board text removed: "ADSR Out"
- board text removed: "Attack"
- board text removed: "CW"
- board text removed: "Decay"
- board text removed: "Gate In"
- board text removed: "JZK Envelope Generator"
- board text removed: "Release"
- board text removed: "Rev. A"
- board text removed: "Sustain"
