File: KiCAD/EG/EG.sch (KiCad schematic (older format))
At the start: 39 parts, among them J1 Power, J2 MJ-3502, J3 MJ-3502, Q1 BC847, Q2 BC847, Q3 BC847, Q4 2N7002, U1 TL074, U2 NE555

Commit message: Added RevB and VCA
Parts:
- added CN1, CN2, CN3, CN4: M3_Screw, Synth:M3_Screw_Hole, symbol Synth:M3_Screw
- C1, C2, C5: Digikey Link (none) -> https://www.digikey.com/short/p4nr3m; Digikey PN (none) -> 720-1540-1-ND; Unit Price (none) -> 0.237
- C3, C4: Digikey Link (none) -> https://www.digikey.com/short/p4nf4h; Digikey PN (none) -> 311-1174-1-ND; Unit Price (none) -> 0.25
- C6: Digikey Link (none) -> https://www.digikey.com/short/p4nf4z; Digikey PN (none) -> 718-1046-1-ND; Unit Price (none) -> 0.70
- D1, D2, D3, D4, D5: footprint Diode_SMD:D_SOD-123 -> Synth:D_SOD-123; Digikey Link (none) -> https://www.digikey.com/short/p4nrm2; Digikey PN (none) -> 1N4148WTPMSCT-ND; Unit Price (none) -> 0.14
- D6: footprint LED_THT:LED_D3.0mm -> Synth:LED_D3.0mm_Clear; Digikey Link (none) -> N/A; Digikey PN (none) -> N/A; Unit Price (none) -> 0.00
- J1: Digikey Link (none) -> https://www.digikey.com/short/p4nr5h; Digikey PN (none) -> 609-3243-ND; Unit Price (none) -> 0.27
- J2, J3: value MJ-3502 -> 4832; footprint Connector_PinHeader_2.54mm:PinHeader_1x02_P2.54mm_Vertical -> Synth:Schurter_4832_Jack; Digikey Link (none) -> https://www.digikey.com/short/p4nr1r; Digikey PN (none) -> 486-3418-ND; Field4 CP-3502MJ-ND -> (none); Field5 None -> (none); Field6 MJ-3502 -> (none); Field7 https://www.cui.com/product/interconnect/connectors/audio-c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 -> (none); Field8 3.5 mm, Mono, Right Angle, Through Hole, Threaded Bushing, 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 -> (none); Field9 CUI Inc. -> (none); Unit Price (none) -> 1.50
- Q1, Q2, Q3: footprint Package_TO_SOT_SMD:SOT-23 -> TO_SOT_Packages_SMD:SOT-23_Handsoldering; Digikey Link (none) -> https://www.digikey.com/short/p4nf4c; Digikey PN (none) -> BC847CLT1GOSCT-ND; Unit Price (none) -> 0.14
- Q4: footprint Package_TO_SOT_SMD:SOT-23 -> TO_SOT_Packages_SMD:SOT-23_Handsoldering; Digikey Link (none) -> https://www.digikey.com/short/p4nf48; Digikey PN (none) -> 2N7002NCT-ND; Unit Price (none) -> 0.39
- R1: Digikey Link (none) -> https://www.digikey.com/short/p4nf4f; Digikey PN (none) -> 311-1.20MFRCT-ND; Unit Price (none) -> 0.10
- R10, R11, R12: Digikey Link (none) -> https://www.digikey.com/short/p4nf40; Digikey PN (none) -> RNCP1206FTD100RCT-ND; Unit Price (none) -> 0.10
- R13, R14: Digikey Link (none) -> https://www.digikey.com/short/p4nrdz; Digikey PN (none) -> 311-1.0KERCT-ND; Unit Price (none) -> 0.10
- R2, R8: Digikey Link (none) -> https://www.digikey.com/short/p4nrn7; Digikey PN (none) -> RMCF1206JT1M00CT-ND; Unit Price (none) -> 0.10
- R3, R5, R6, R7: Digikey Link (none) -> https://www.digikey.com/short/p4nr22; Digikey PN (none) -> A130554CT-ND; Unit Price (none) -> 0.33
- R4: Digikey Link (none) -> https://www.digikey.com/short/p4nrn9; Digikey PN (none) -> P10ALCT-ND; Unit Price (none) -> 0.17
- R9: Digikey Link (none) -> https://www.digikey.com/short/p4nr81; Digikey PN (none) -> A130181CT-ND; Unit Price (none) -> 0.10
- RV1: footprint Connector_PinHeader_2.54mm:PinHeader_1x03_P2.54mm_Vertical -> Synth:Potentiometer_Bourns_PTV09A-1_Single_Vertical; Digikey Link (none) -> https://www.digikey.com/short/p4nfq1; Digikey PN (none) -> PTV09A-4020F-B203-ND; Unit Price (none) -> 0.83
- RV2, RV3, RV4: footprint Connector_PinHeader_2.54mm:PinHeader_1x03_P2.54mm_Vertical -> Synth:Potentiometer_Bourns_PTV09A-1_Single_Vertical; Digikey Link (none) -> https://www.digikey.com/short/p4nfhw; Digikey PN (none) -> PTV09A-4020F-A504-ND; Unit Price (none) -> 0.83
- U1: Digikey Link (none) -> https://www.digikey.com/short/p4nrh2; Digikey PN (none) -> 296-1283-1-ND; Unit Price (none) -> 0.60
- U2: Digikey Link (none) -> https://www.digikey.com/short/p4nfzd; Digikey PN (none) -> 296-6501-1-ND; Unit Price (none) -> 0.48
Connections:
- net at Q4.3 (D): now also RV1.1; no longer RV1.3
- net at R9.2: now also RV1.3; no longer RV1.1
- net Sustain: now reaches RV1.2, U1.3 (+)
- net Decay: now reaches R12.1, RV4.2
- net Attack: now reaches R11.2, RV2.2
- net Release: now reaches R10.2, RV3.2
Other:
- note removed: "Attack"
- note removed: "Decay"
- note removed: "Release"
- note removed: "Sustain"
