File: KiCAD/MIDI Controller/MIDI Controller.kicad_pcb (KiCad board)
At the start: 2 copper layers, 90 x 80 mm, 81 parts, among them J1 2040002-1, J10 MJ-3502, J11 MJ-3502, J12 MJ-3502, J13 MJ-3502, J14 MJ-3502, J15 MJ-3502, J16 MJ-3502, J17 MJ-3502, J2 Power, J3 MIDI, J4 Prog Jumper, J5 MJ-3502, J6 MJ-3502, J7 MJ-3502, J8 MJ-3502, J9 MJ-3502, U1 ATmega328PB-AU, U10 AD5293, U11 6N138, U12 TL074, U13 TL074, U14 TL074, U15 TL074, U2 FT232RL, U3 AD5293, U4 AD5293, U5 AD5293, U6 LM1117-5.0, U7 AD5293, U8 AD5293, U9 AD5293, Y1 16 MHz

Commit message: Added MIDI controller and PSU
Parts:
- removed C1, C2, C6: 0.1uF, Synth:C_1206
- removed C16, C3, C5: 1uF, Synth:C_1206
- removed C4: 4.7uF, Synth:C_1206
- removed J1: 2040002-1, Synth:2040002
- removed R1, R2, R3: 1k, Synth:R_1206
- removed the REF** at (65.0, 125.0)
- removed the REF** at (145.0, 125.0)
- removed the REF** at (145.0, 55.0)
- removed the REF** at (65.0, 55.0)
- removed U1: ATmega328PB-AU, Package_QFP:TQFP-32_7x7mm_P0.8mm
- removed U2: FT232RL, Package_SO:SSOP-28_5.3x10.2mm_P0.65mm
- removed U6: LM1117-5.0, Package_TO_SOT_SMD:SOT-223-3_TabPin2
- removed Y1: 16 MHz, Synth:Abracon_AWSCR_4.7x4.1mm
- added A1: Arduino_Nano_v3.x, Module:Arduino_Nano, F.Cu at (79.4, 51.9)
- added REF**: CUI_SD-50SN_PCB, Synth:CUI_SD-50SN_PCB, F.Cu at (70.0, 110.0)
- added SC1: M3_Screw_Hole, Synth:M3_Screw_Hole, F.Cu at (45.0, 35.0)
- added SC2: M3_Screw_Hole, Synth:M3_Screw_Hole, F.Cu at (115.0, 35.0)
- added SC3: M3_Screw_Hole, Synth:M3_Screw_Hole, F.Cu at (45.0, 125.0)
- added SC4: M3_Screw_Hole, Synth:M3_Screw_Hole, F.Cu at (115.0, 125.0)
- D1: value 1N914 -> 1N4148W; footprint Diode_THT:D_DO-35_SOD27_P7.62mm_Horizontal -> Synth:D_SOD-123
- J10, J11, J12, J13, J14, J15, J16, J17, J5, J6, J7, J8, J9: value MJ-3502 -> 4832; footprint Connector_PinHeader_2.54mm:PinHeader_1x02_P2.54mm_Vertical -> Synth:Schurter_4832_Jack; moved to B.Cu
- moved C33 85.1 mm to (77.4, 34.4), turned to 0 degrees
- moved C31 82.1 mm to (65.8, 34.4), turned to 0 degrees
- moved C35 78.4 mm to (93.2, 41.3), turned to 270 degrees
- moved C36 76.9 mm to (86.9, 32.9)
- moved U15 76.6 mm to (86.7, 39.3)
- moved U13 74.4 mm to (63.8, 40.1), turned to 270 degrees
- moved U14 73.4 mm to (75.4, 40.1), turned to 270 degrees
- moved C29 71.6 mm to (54.3, 34.4), turned to 0 degrees
- moved J3 71.4 mm to (79.7, 119.5), turned to 0 degrees
- moved J17 70.4 mm to (50.0, 110.0)
- moved R4 67.7 mm to (85.5, 122.1), turned to 0 degrees
- moved C32 66.2 mm to (62.0, 48.1), turned to 90 degrees
- moved J10 64.6 mm to (60.0, 65.0), turned to 180 degrees
- moved J11 63.0 mm to (50.0, 65.0), turned to 180 degrees
- moved U12 61.9 mm to (52.3, 40.1), turned to 270 degrees
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Connections:
- J10 pad 2: Net-(J10-Pad2) -> /External Pins/Velocity2
- J11 pad 2: Net-(J11-Pad2) -> /External Pins/Trig2
- J12 pad 2: Net-(J12-Pad2) -> /External Pins/Clock2
- J13 pad 2: Net-(J13-Pad2) -> /External Pins/Note3
- J14 pad 2: Net-(J14-Pad2) -> /External Pins/Velocity3
- J15 pad 2: Net-(J15-Pad2) -> /External Pins/Trig3
- J16 pad 2: Net-(J16-Pad2) -> /External Pins/Clock4
- J17 pad 2: Net-(J17-Pad2) -> /External Pins/Aftertouch
- J4 pad 2: Prog_Rx -> Net-(A1-Pad2)
- J5 pad 2: Net-(J5-Pad2) -> /External Pins/Note1
- J6 pad 2: Net-(J6-Pad2) -> /External Pins/Velocity1
- J7 pad 2: Net-(J7-Pad2) -> /External Pins/Trig1
- J8 pad 2: Net-(J8-Pad2) -> /External Pins/Clock1
- J9 pad 2: Net-(J9-Pad2) -> /External Pins/Note2
- U12 pad 1: Net-(J5-Pad2) -> /External Pins/Note1
- U12 pad 13: Net-(J8-Pad2) -> /External Pins/Clock1
- U12 pad 14: Net-(J8-Pad2) -> /External Pins/Clock1
- U12 pad 2: Net-(J5-Pad2) -> /External Pins/Note1
- U12 pad 6: Net-(J6-Pad2) -> /External Pins/Velocity1
- U12 pad 7: Net-(J6-Pad2) -> /External Pins/Velocity1
- U12 pad 8: Net-(J7-Pad2) -> /External Pins/Trig1
- U12 pad 9: Net-(J7-Pad2) -> /External Pins/Trig1
- U13 pad 1: Net-(J9-Pad2) -> /External Pins/Note2
- U13 pad 13: Net-(J12-Pad2) -> /External Pins/Clock2
- U13 pad 14: Net-(J12-Pad2) -> /External Pins/Clock2
- U13 pad 2: Net-(J9-Pad2) -> /External Pins/Note2
- U13 pad 6: Net-(J10-Pad2) -> /External Pins/Velocity2
- U13 pad 7: Net-(J10-Pad2) -> /External Pins/Velocity2
- U13 pad 8: Net-(J11-Pad2) -> /External Pins/Trig2
- U13 pad 9: Net-(J11-Pad2) -> /External Pins/Trig2
- U14 pad 1: Net-(J13-Pad2) -> /External Pins/Note3
- U14 pad 13: Net-(J16-Pad2) -> /External Pins/Clock4
- U14 pad 14: Net-(J16-Pad2) -> /External Pins/Clock4
- U14 pad 2: Net-(J13-Pad2) -> /External Pins/Note3
- U14 pad 6: Net-(J14-Pad2) -> /External Pins/Velocity3
- U14 pad 7: Net-(J14-Pad2) -> /External Pins/Velocity3
- U14 pad 8: Net-(J15-Pad2) -> /External Pins/Trig3
- U14 pad 9: Net-(J15-Pad2) -> /External Pins/Trig3
- U15 pad 1: Net-(J17-Pad2) -> /External Pins/Aftertouch
- U15 pad 2: Net-(J17-Pad2) -> /External Pins/Aftertouch
Routing:
- net +5V: track 292.1 -> 159.6 mm
- net /External Pins/Aftertouch: track 0.00 -> 94.8 mm
- net +12V: track 165.5 -> 73.8 mm, vias 17 -> 21
- net CV2: track 15.4 -> 99.0 mm, vias 0 -> 2
- net /External Pins/Clock4: track 0.00 -> 82.4 mm
- net /External Pins/Clock1: track 0.00 -> 74.2 mm
- net Net-(J1-Pad2): track 73.7 -> 0.00 mm
- net Net-(J1-Pad3): track 73.6 -> 0.00 mm
- net -12V: track 234.2 -> 302.7 mm, vias 4 -> 0
- net /External Pins/Clock2: track 0.00 -> 66.4 mm
- net GND: track 120.5 -> 182.2 mm, vias 35 -> 28
- net CV7: track 16.1 -> 76.1 mm
- net CV5: track 15.6 -> 73.4 mm, vias 0 -> 2
- net /External Pins/Trig3: track 0.00 -> 57.2 mm
- net CV4: track 15.5 -> 71.2 mm
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- added copper zone on B.Cu, net +12V
- added copper zone on F.Cu, net GND
- removed copper zone on F.Cu, net +12V
- removed copper zone on B.Cu, net GND
Other:
- board size 90 x 80 mm -> 80 x 100 mm
- board text added: "5 4"
- board text added: "AFTERTOUCH"
- board text added: "ARDUINO NANO"
- board text added: "CLOCK 1"
- board text added: "CLOCK 2"
- board text added: "CLOCK 4"
- board text added: "JZK MIDI CONTROLLER Rev B"
- board text added: "Jonathan Kayne Virginia Tech ECE"
- board text added: "NOTE 1"
- board text added: "NOTE 2"
- board text added: "NOTE 3"
- board text added: "TRIG 1"
- board text added: "TRIG 2"
- board text added: "TRIG 3"
- board text added: "VEL 1"
- board text added: "VEL 2"
- board text added: "VEL 3"
- board text removed: "2 4"
- board text removed: "Aftertouch"
- board text removed: "Clock 1"
- board text removed: "Clock 2"
- board text removed: "Clock 4"
- board text removed: "JZK MIDI CONTROLLER"
- board text removed: "Jonathan Kayne 2019 Virginia Tech ECE"
- board text removed: "Note 1"
- board text removed: "Note 2"
- board text removed: "Note 3"
- board text removed: "Rev. A"
- board text removed: "Trig 1"
- board text removed: "Trig 2"
- board text removed: "Trig 3"
- board text removed: "Vel 1"
- board text removed: "Vel 2"
- board text removed: "Vel 3"
